Commit message: updated everything for the fake parts added

File: robot_moveit_config/config/spotarm_assembly.ros2_control.xacro (robot description, xacro)
@@ -43,4 +43,11 @@
                 <state_interface name="velocity"/>
             </joint>
+            <joint name="Revolute6">
+                <command_interface name="position"/>
+                <state_interface name="position">
+                  <param name="initial_value">${initial_positions['Revolute6']}</param>
+                </state_interface>
+                <state_interface name="velocity"/>
+            </joint>
         </ros2_control>
     </xacro:macro>

File: spotarm_assembly_description/urdf/spotarm_assembly.ros2_control.xacro (robot description, xacro)
@@ -41,4 +41,11 @@
           <state_interface name="velocity"/>
       </joint>
+      <joint name="Revolute6">
+          <command_interface name="position"/>
+          <state_interface name="position">
+            <param name="initial_value">0.0</param>
+          </state_interface>
+          <state_interface name="velocity"/>
+      </joint>
   </ros2_control>
 </robot>

File: spotarm_assembly_description/urdf/spotarm_assembly.urdf (robot description, URDF)
Before this commit: robot spotarm_assembly, 6 links, 5 joints
Links:
- removed link stub_link
- added link fake_gripper, mass 0.05; collision box size=0.04 0.08 0.04; visual box size=0.01 0.06 0.01
- added link link_6_fake, mass 0.2; collision box size=0.02 0.2 0.02; visual box size=0.02 0.2 0.02
- added link link_7_fake, mass 0.2; collision box size=0.02 0.2 0.02; visual box size=0.02 0.1 0.02
Joints:
- added joint Revolute6: type continuous, parent link_6_fake, child link_7_fake, origin xyz=0.011 -0.19 0 rpy=0 0 0, axis 0.0 1.0 0.0
- added joint fake_gripper_fixed: type fixed, parent link_7_fake, child fake_gripper, origin xyz=0 -0.1 0 rpy=0 0 0
- joint Revolute5: child stub_link -> link_6_fake
