Commit message: Updated LED code to properly work on the Arm Added PWM output node for the end effector Still a little shakey due to math and PWM timing inaccuracies

File: build/spotarm_assembly_description/urdf/materials.xacro (robot description, xacro)
@@ -1 +1 @@
-/home/msd/MSD2/REV4/src/spotarm_assembly_description/urdf/materials.xacro
+/mnt/c/Users/Oden2/Downloads/MSD-SPOT-robot-Rev-4/src/spotarm_assembly_description/urdf/materials.xacro

File: build/spotarm_assembly_description/urdf/spotarm_assembly.ros2_control.xacro (robot description, xacro)
@@ -1 +1 @@
-/home/msd/MSD2/REV4/src/spotarm_assembly_description/urdf/spotarm_assembly.ros2_control.xacro
+/mnt/c/Users/Oden2/Downloads/MSD-SPOT-robot-Rev-4/src/spotarm_assembly_description/urdf/spotarm_assembly.ros2_control.xacro

File: build/spotarm_assembly_description/urdf/spotarm_assembly.xacro (robot description, xacro)
@@ -1 +1 @@
-/home/msd/MSD2/REV4/src/spotarm_assembly_description/urdf/spotarm_assembly.xacro
+/mnt/c/Users/Oden2/Downloads/MSD-SPOT-robot-Rev-4/src/spotarm_assembly_description/urdf/spotarm_assembly.xacro

File: install/gear_manipulator_moveit_config/share/gear_manipulator_moveit_config/config/gear_manipulator.ros2_control.xacro (robot description, xacro)
@@ -1,47 +1 @@
-<?xml version="1.0"?>
-<robot xmlns:xacro="http://www.ros.org/wiki/xacro">
-    <xacro:macro name="gear_manipulator_ros2_control" params="name initial_positions_file">
-        <xacro:property name="initial_positions" value="${load_yaml(initial_positions_file)['initial_positions']}"/>
-        <ros2_control name="${name}" type="system">
-            <hardware>
-                <!-- By default, set up controllers for simulation. This won't work on real hardware -->
-                <plugin>mock_components/GenericSystem</plugin>
-            </hardware>
-            <joint name="joint1">
-                <command_interface name="position"/>
-                <state_interface name="position">
-                  <param name="initial_value">${initial_positions['joint1']}</param>
-                </state_interface>
-                <state_interface name="velocity"/>
-            </joint>
-            <joint name="joint2">
-                <command_interface name="position"/>
-                <state_interface name="position">
-                  <param name="initial_value">${initial_positions['joint2']}</param>
-                </state_interface>
-                <state_interface name="velocity"/>
-            </joint>
-            <joint name="joint3">
-                <command_interface name="position"/>
-                <state_interface name="position">
-                  <param name="initial_value">${initial_positions['joint3']}</param>
-                </state_interface>
-                <state_interface name="velocity"/>
-            </joint>
-            <joint name="joint4">
-                <command_interface name="position"/>
-                <state_interface name="position">
-                  <param name="initial_value">${initial_positions['joint4']}</param>
-                </state_interface>
-                <state_interface name="velocity"/>
-            </joint>
-            <joint name="joint5">
-                <command_interface name="position"/>
-                <state_interface name="position">
-                  <param name="initial_value">${initial_positions['joint5']}</param>
-                </state_interface>
-                <state_interface name="velocity"/>
-            </joint>
-        </ros2_control>
-    </xacro:macro>
-</robot>
+/mnt/c/Users/Oden2/Downloads/MSD-SPOT-robot-Rev-4/src/gear_manipulator_moveit_config/config/gear_manipulator.ros2_control.xacro

File: install/gear_manipulator_moveit_config/share/gear_manipulator_moveit_config/config/gear_manipulator.urdf.xacro (robot description, xacro)
@@ -1,9 +1 @@
-<?xml version="1.0"?>
-<robot xmlns:xacro="http://www.ros.org/wiki/xacro" name="gear_manipulator">
-    <xacro:arg name="initial_positions_file" default="initial_positions.yaml" />
-    <!-- Import gear_manipulator urdf file -->
-    <xacro:include filename="$(find my_robot)/urdf/gear_manipulator.urdf" />
-    <!-- Import control_xacro -->
-    <xacro:include filename="gear_manipulator.ros2_control.xacro" />
-    <xacro:gear_manipulator_ros2_control name="FakeSystem" initial_positions_file="$(arg initial_positions_file)"/>
-</robot>
+/mnt/c/Users/Oden2/Downloads/MSD-SPOT-robot-Rev-4/src/gear_manipulator_moveit_config/config/gear_manipulator.urdf.xacro

File: install/robot_moveit_config/share/robot_moveit_config/config/spotarm_assembly.hardware.urdf.xacro (robot description, xacro)
@@ -1 +1 @@
-/home/msd/MSD2/REV4/src/robot_moveit_config/config/spotarm_assembly.hardware.urdf.xacro
+/mnt/c/Users/Oden2/Downloads/MSD-SPOT-robot-Rev-4/src/robot_moveit_config/config/spotarm_assembly.hardware.urdf.xacro

File: install/robot_moveit_config/share/robot_moveit_config/config/spotarm_assembly.ros2_control.xacro (robot description, xacro)
@@ -1 +1 @@
-/home/msd/MSD2/REV4/src/robot_moveit_config/config/spotarm_assembly.ros2_control.xacro
+/mnt/c/Users/Oden2/Downloads/MSD-SPOT-robot-Rev-4/src/robot_moveit_config/config/spotarm_assembly.ros2_control.xacro

File: install/robot_moveit_config/share/robot_moveit_config/config/spotarm_assembly.urdf.xacro (robot description, xacro)
@@ -1 +1 @@
-/home/msd/MSD2/REV4/src/robot_moveit_config/config/spotarm_assembly.urdf.xacro
+/mnt/c/Users/Oden2/Downloads/MSD-SPOT-robot-Rev-4/src/robot_moveit_config/config/spotarm_assembly.urdf.xacro

File: install/spotarm_assembly_description/share/spotarm_assembly_description/urdf/materials.xacro (robot description, xacro)
@@ -1 +1 @@
-/home/msd/MSD2/REV4/build/spotarm_assembly_description/urdf/materials.xacro
+/mnt/c/Users/Oden2/Downloads/MSD-SPOT-robot-Rev-4/build/spotarm_assembly_description/urdf/materials.xacro

File: install/spotarm_assembly_description/share/spotarm_assembly_description/urdf/spotarm_assembly.ros2_control.xacro (robot description, xacro)
@@ -1 +1 @@
-/home/msd/MSD2/REV4/build/spotarm_assembly_description/urdf/spotarm_assembly.ros2_control.xacro
+/mnt/c/Users/Oden2/Downloads/MSD-SPOT-robot-Rev-4/build/spotarm_assembly_description/urdf/spotarm_assembly.ros2_control.xacro

File: install/spotarm_assembly_description/share/spotarm_assembly_description/urdf/spotarm_assembly.xacro (robot description, xacro)
@@ -1 +1 @@
-/home/msd/MSD2/REV4/build/spotarm_assembly_description/urdf/spotarm_assembly.xacro
+/mnt/c/Users/Oden2/Downloads/MSD-SPOT-robot-Rev-4/build/spotarm_assembly_description/urdf/spotarm_assembly.xacro

Commit message: Added good end effector code.

File: build/spotarm_assembly_description/urdf/materials.xacro (robot description, xacro)
@@ -1 +1 @@
-/mnt/c/Users/Oden2/Downloads/MSD-SPOT-robot-Rev-4/src/spotarm_assembly_description/urdf/materials.xacro
+/home/msd/MSD2/REV4/src/spotarm_assembly_description/urdf/materials.xacro

File: build/spotarm_assembly_description/urdf/spotarm_assembly.ros2_control.xacro (robot description, xacro)
@@ -1 +1 @@
-/mnt/c/Users/Oden2/Downloads/MSD-SPOT-robot-Rev-4/src/spotarm_assembly_description/urdf/spotarm_assembly.ros2_control.xacro
+/home/msd/MSD2/REV4/src/spotarm_assembly_description/urdf/spotarm_assembly.ros2_control.xacro

File: build/spotarm_assembly_description/urdf/spotarm_assembly.xacro (robot description, xacro)
@@ -1 +1 @@
-/mnt/c/Users/Oden2/Downloads/MSD-SPOT-robot-Rev-4/src/spotarm_assembly_description/urdf/spotarm_assembly.xacro
+/home/msd/MSD2/REV4/src/spotarm_assembly_description/urdf/spotarm_assembly.xacro

File: install/gear_manipulator_moveit_config/share/gear_manipulator_moveit_config/config/gear_manipulator.ros2_control.xacro (robot description, xacro)
@@ -1 +1,47 @@
-/mnt/c/Users/Oden2/Downloads/MSD-SPOT-robot-Rev-4/src/gear_manipulator_moveit_config/config/gear_manipulator.ros2_control.xacro
+<?xml version="1.0"?>
+<robot xmlns:xacro="http://www.ros.org/wiki/xacro">
+    <xacro:macro name="gear_manipulator_ros2_control" params="name initial_positions_file">
+        <xacro:property name="initial_positions" value="${load_yaml(initial_positions_file)['initial_positions']}"/>
+        <ros2_control name="${name}" type="system">
+            <hardware>
+                <!-- By default, set up controllers for simulation. This won't work on real hardware -->
+                <plugin>mock_components/GenericSystem</plugin>
+            </hardware>
+            <joint name="joint1">
+                <command_interface name="position"/>
+                <state_interface name="position">
+                  <param name="initial_value">${initial_positions['joint1']}</param>
+                </state_interface>
+                <state_interface name="velocity"/>
+            </joint>
+            <joint name="joint2">
+                <command_interface name="position"/>
+                <state_interface name="position">
+                  <param name="initial_value">${initial_positions['joint2']}</param>
+                </state_interface>
+                <state_interface name="velocity"/>
+            </joint>
+            <joint name="joint3">
+                <command_interface name="position"/>
+                <state_interface name="position">
+                  <param name="initial_value">${initial_positions['joint3']}</param>
+                </state_interface>
+                <state_interface name="velocity"/>
+            </joint>
+            <joint name="joint4">
+                <command_interface name="position"/>
+                <state_interface name="position">
+                  <param name="initial_value">${initial_positions['joint4']}</param>
+                </state_interface>
+                <state_interface name="velocity"/>
+            </joint>
+            <joint name="joint5">
+                <command_interface name="position"/>
+                <state_interface name="position">
+                  <param name="initial_value">${initial_positions['joint5']}</param>
+                </state_interface>
+                <state_interface name="velocity"/>
+            </joint>
+        </ros2_control>
+    </xacro:macro>
+</robot>

File: install/gear_manipulator_moveit_config/share/gear_manipulator_moveit_config/config/gear_manipulator.urdf.xacro (robot description, xacro)
@@ -1 +1,9 @@
-/mnt/c/Users/Oden2/Downloads/MSD-SPOT-robot-Rev-4/src/gear_manipulator_moveit_config/config/gear_manipulator.urdf.xacro
+<?xml version="1.0"?>
+<robot xmlns:xacro="http://www.ros.org/wiki/xacro" name="gear_manipulator">
+    <xacro:arg name="initial_positions_file" default="initial_positions.yaml" />
+    <!-- Import gear_manipulator urdf file -->
+    <xacro:include filename="$(find my_robot)/urdf/gear_manipulator.urdf" />
+    <!-- Import control_xacro -->
+    <xacro:include filename="gear_manipulator.ros2_control.xacro" />
+    <xacro:gear_manipulator_ros2_control name="FakeSystem" initial_positions_file="$(arg initial_positions_file)"/>
+</robot>

File: install/robot_moveit_config/share/robot_moveit_config/config/spotarm_assembly.hardware.urdf.xacro (robot description, xacro)
@@ -1 +1 @@
-/mnt/c/Users/Oden2/Downloads/MSD-SPOT-robot-Rev-4/src/robot_moveit_config/config/spotarm_assembly.hardware.urdf.xacro
+/home/msd/MSD2/REV4/src/robot_moveit_config/config/spotarm_assembly.hardware.urdf.xacro

File: install/robot_moveit_config/share/robot_moveit_config/config/spotarm_assembly.ros2_control.xacro (robot description, xacro)
@@ -1 +1 @@
-/mnt/c/Users/Oden2/Downloads/MSD-SPOT-robot-Rev-4/src/robot_moveit_config/config/spotarm_assembly.ros2_control.xacro
+/home/msd/MSD2/REV4/src/robot_moveit_config/config/spotarm_assembly.ros2_control.xacro

File: install/robot_moveit_config/share/robot_moveit_config/config/spotarm_assembly.urdf.xacro (robot description, xacro)
@@ -1 +1 @@
-/mnt/c/Users/Oden2/Downloads/MSD-SPOT-robot-Rev-4/src/robot_moveit_config/config/spotarm_assembly.urdf.xacro
+/home/msd/MSD2/REV4/src/robot_moveit_config/config/spotarm_assembly.urdf.xacro

File: install/spotarm_assembly_description/share/spotarm_assembly_description/urdf/materials.xacro (robot description, xacro)
@@ -1 +1 @@
-/mnt/c/Users/Oden2/Downloads/MSD-SPOT-robot-Rev-4/build/spotarm_assembly_description/urdf/materials.xacro
+/home/msd/MSD2/REV4/build/spotarm_assembly_description/urdf/materials.xacro

File: install/spotarm_assembly_description/share/spotarm_assembly_description/urdf/spotarm_assembly.ros2_control.xacro (robot description, xacro)
@@ -1 +1 @@
-/mnt/c/Users/Oden2/Downloads/MSD-SPOT-robot-Rev-4/build/spotarm_assembly_description/urdf/spotarm_assembly.ros2_control.xacro
+/home/msd/MSD2/REV4/build/spotarm_assembly_description/urdf/spotarm_assembly.ros2_control.xacro

File: install/spotarm_assembly_description/share/spotarm_assembly_description/urdf/spotarm_assembly.xacro (robot description, xacro)
@@ -1 +1 @@
-/mnt/c/Users/Oden2/Downloads/MSD-SPOT-robot-Rev-4/build/spotarm_assembly_description/urdf/spotarm_assembly.xacro
+/home/msd/MSD2/REV4/build/spotarm_assembly_description/urdf/spotarm_assembly.xacro
