Commit message: Working Crued Endeffector

File: install/gear_manipulator_moveit_config/share/gear_manipulator_moveit_config/config/gear_manipulator.ros2_control.xacro (robot description, xacro)
@@ -1 +1,47 @@
-/home/msd/MSD2/REV4/src/gear_manipulator_moveit_config/config/gear_manipulator.ros2_control.xacro
+<?xml version="1.0"?>
+<robot xmlns:xacro="http://www.ros.org/wiki/xacro">
+    <xacro:macro name="gear_manipulator_ros2_control" params="name initial_positions_file">
+        <xacro:property name="initial_positions" value="${load_yaml(initial_positions_file)['initial_positions']}"/>
+        <ros2_control name="${name}" type="system">
+            <hardware>
+                <!-- By default, set up controllers for simulation. This won't work on real hardware -->
+                <plugin>mock_components/GenericSystem</plugin>
+            </hardware>
+            <joint name="joint1">
+                <command_interface name="position"/>
+                <state_interface name="position">
+                  <param name="initial_value">${initial_positions['joint1']}</param>
+                </state_interface>
+                <state_interface name="velocity"/>
+            </joint>
+            <joint name="joint2">
+                <command_interface name="position"/>
+                <state_interface name="position">
+                  <param name="initial_value">${initial_positions['joint2']}</param>
+                </state_interface>
+                <state_interface name="velocity"/>
+            </joint>
+            <joint name="joint3">
+                <command_interface name="position"/>
+                <state_interface name="position">
+                  <param name="initial_value">${initial_positions['joint3']}</param>
+                </state_interface>
+                <state_interface name="velocity"/>
+            </joint>
+            <joint name="joint4">
+                <command_interface name="position"/>
+                <state_interface name="position">
+                  <param name="initial_value">${initial_positions['joint4']}</param>
+                </state_interface>
+                <state_interface name="velocity"/>
+            </joint>
+            <joint name="joint5">
+                <command_interface name="position"/>
+                <state_interface name="position">
+                  <param name="initial_value">${initial_positions['joint5']}</param>
+                </state_interface>
+                <state_interface name="velocity"/>
+            </joint>
+        </ros2_control>
+    </xacro:macro>
+</robot>

File: install/gear_manipulator_moveit_config/share/gear_manipulator_moveit_config/config/gear_manipulator.urdf.xacro (robot description, xacro)
@@ -1 +1,9 @@
-/home/msd/MSD2/REV4/src/gear_manipulator_moveit_config/config/gear_manipulator.urdf.xacro
+<?xml version="1.0"?>
+<robot xmlns:xacro="http://www.ros.org/wiki/xacro" name="gear_manipulator">
+    <xacro:arg name="initial_positions_file" default="initial_positions.yaml" />
+    <!-- Import gear_manipulator urdf file -->
+    <xacro:include filename="$(find my_robot)/urdf/gear_manipulator.urdf" />
+    <!-- Import control_xacro -->
+    <xacro:include filename="gear_manipulator.ros2_control.xacro" />
+    <xacro:gear_manipulator_ros2_control name="FakeSystem" initial_positions_file="$(arg initial_positions_file)"/>
+</robot>

Commit message: Working Joystick

File: install/gear_manipulator_moveit_config/share/gear_manipulator_moveit_config/config/gear_manipulator.ros2_control.xacro (robot description, xacro)
@@ -1,47 +1 @@
-<?xml version="1.0"?>
-<robot xmlns:xacro="http://www.ros.org/wiki/xacro">
-    <xacro:macro name="gear_manipulator_ros2_control" params="name initial_positions_file">
-        <xacro:property name="initial_positions" value="${load_yaml(initial_positions_file)['initial_positions']}"/>
-        <ros2_control name="${name}" type="system">
-            <hardware>
-                <!-- By default, set up controllers for simulation. This won't work on real hardware -->
-                <plugin>mock_components/GenericSystem</plugin>
-            </hardware>
-            <joint name="joint1">
-                <command_interface name="position"/>
-                <state_interface name="position">
-                  <param name="initial_value">${initial_positions['joint1']}</param>
-                </state_interface>
-                <state_interface name="velocity"/>
-            </joint>
-            <joint name="joint2">
-                <command_interface name="position"/>
-                <state_interface name="position">
-                  <param name="initial_value">${initial_positions['joint2']}</param>
-                </state_interface>
-                <state_interface name="velocity"/>
-            </joint>
-            <joint name="joint3">
-                <command_interface name="position"/>
-                <state_interface name="position">
-                  <param name="initial_value">${initial_positions['joint3']}</param>
-                </state_interface>
-                <state_interface name="velocity"/>
-            </joint>
-            <joint name="joint4">
-                <command_interface name="position"/>
-                <state_interface name="position">
-                  <param name="initial_value">${initial_positions['joint4']}</param>
-                </state_interface>
-                <state_interface name="velocity"/>
-            </joint>
-            <joint name="joint5">
-                <command_interface name="position"/>
-                <state_interface name="position">
-                  <param name="initial_value">${initial_positions['joint5']}</param>
-                </state_interface>
-                <state_interface name="velocity"/>
-            </joint>
-        </ros2_control>
-    </xacro:macro>
-</robot>
+/home/msd/MSD2/REV4/src/gear_manipulator_moveit_config/config/gear_manipulator.ros2_control.xacro

File: install/gear_manipulator_moveit_config/share/gear_manipulator_moveit_config/config/gear_manipulator.urdf.xacro (robot description, xacro)
@@ -1,9 +1 @@
-<?xml version="1.0"?>
-<robot xmlns:xacro="http://www.ros.org/wiki/xacro" name="gear_manipulator">
-    <xacro:arg name="initial_positions_file" default="initial_positions.yaml" />
-    <!-- Import gear_manipulator urdf file -->
-    <xacro:include filename="$(find my_robot)/urdf/gear_manipulator.urdf" />
-    <!-- Import control_xacro -->
-    <xacro:include filename="gear_manipulator.ros2_control.xacro" />
-    <xacro:gear_manipulator_ros2_control name="FakeSystem" initial_positions_file="$(arg initial_positions_file)"/>
-</robot>
+/home/msd/MSD2/REV4/src/gear_manipulator_moveit_config/config/gear_manipulator.urdf.xacro
